File: eagle/Circuits.sch (EAGLE design)
At the start: 33 parts, among them IC1 74AC14N, IC2 74AC14N, IC3 74AC14N, IC4 74AC14N, IC5 PCF8574P, IC6 MCP603

Commit message: everything's dandy with electronics
Parts:
- removed IC3, IC4: 74AC14N, 74xx-eu:74AC14N
- removed IC6: MCP603, maxim:MAX4105EUK
- removed LED4: LAW57B, led:LAW57B
- added LED6: TLLR4400, led:TLLR4400
- added R15: 220, resistor:R-EU_0207/7
- added X1: JP1, con-molex:22-23-2041
- D2: device opto-trans-siemens:BPW32 -> opto-trans-siemens:SFH205
- IC2: value 74AC14N -> mcp603; device 74xx-eu:74AC14N -> analog-devices:AD811N
- JP4: value M05X2SHD -> Prog-Header
- LED1, LED2, LED3: value LAW57B -> TLLR4400; device led:LAW57B -> led:TLLR4400
- R13: device resistor:R-EU_0207/7 -> resistor:R-EU_0204/5
Connections:
- new net N$20: D1.CATHODE, R15.2
- new net N$21: U$1.(PCINT10/INT0/OC0A/CKOUT)PB2, X1-1.S
- net +5V: now also IC1P.VCC, IC2.+VS, LED6.A; no longer LED4.A
- net COLOUR-1: no longer U$1.(PCINT10/INT0/OC0A/CKOUT)PB2
- net COLOUR-2: now also X1-3.S
- net COLOUR-3: now also X1-4.S
- net GND: now also IC1P.GND, IC2.-VS, IC2.IN+, R15.1, X1-2.S; no longer D1.CATHODE, IC6G$1.+IN
- net LINE2: now also IC1B.O; no longer IC2A.O
- net LINE3: now also IC1C.O; no longer IC3A.O
- net LINE4: now also IC1D.O; no longer IC4A.O
- net N$13: now also IC1D.I; no longer IC4A.I
- net N$16: now also LED6.C; no longer LED4.C
- net N$19: now also IC2.IN-; no longer IC6G$1.-IN
- net N$5: now also IC1B.I; no longer IC2A.I
- net N$9: now also IC1C.I; no longer IC3A.I
- net PHOTO_OUT: now also IC2.OUT, U$1.(PCINT3/T0/ADC3)PA3; no longer IC6G$1.OUT, U$1.(PCINT7/ICP/OC0B/ADC7)PA7
Other:
- note added: "SCK"
- note added: "SDA"
- note removed: "SCK out"
- note removed: "SDA out"
- moved on the sheet: C1, D2, R13

Commit message: Added PIC colour sensor as DA Backup
Parts:
- added C3: 16pF, resistor:C-EU025-024X044
- added C4: 22pF, resistor:C-EU025-024X044
- added D3: LED-RGB-CC-THRUCLEAR, SparkFun-LED:LED-RGB-CC-THRUCLEAR
- added D4: SFH213, opto-trans-siemens:SFH205
- added IC4: mcp603, analog-devices:AD811N
- added IC6: PIC12F675P, microchip:PIC12F675P
- added JP5: (no value), SparkFun-Connectors:M04LONGPADS
- added JP6: (no value), SparkFun-Connectors:M05PTH_LONGPADS
- added R16: 1M, resistor:R-EU_0204/5
- added R17, R21: 10k, resistor:R-EU_0207/7
- added R18, R19, R20: 220, resistor:R-EU_0207/7
Connections:
- removed net N$21: U$1.(PCINT10/INT0/OC0A/CKOUT)PB2, X1-1.S
- new net N$22: D3.BLUE_CATHODE, R18.1
- new net N$23: D3.GREEN_CATHODE, R19.1
- new net N$24: IC6.GP5/CLKIN, R17.2
- new net N$25: C3.1, D4.A, IC4.IN-, R16.1
- new net N$28: D3.RED_CATHODE, R20.1
- new net N$29: IC6.GP2/AN2, R18.2
- new net PROG-CLK: IC6.VREF/GP1/AN1, JP6.3, R19.2
- new net PROG-IO: IC6.GP0/AN0, JP6.4, R20.2
- new net VPP: IC6.GP3/!MCLR, JP6.2, R21.1
- net +5V: now also C4.2, IC4.+VS, IC6.VCC, JP5.1, JP6.1
- net COLOUR-1: now also JP5.3, R21.2, U$1.(PCINT10/INT0/OC0A/CKOUT)PB2, X1-1.S
- net COLOUR-2: now also JP5.2, R17.1
- net GND: now also C4.1, D3.CATHODE, D4.C, IC4.-VS, IC4.IN+, IC6.GND, JP5.4, JP6.5
- net PHOTO_OUT: now also C3.2, IC4.OUT, IC6.GP4/AN3, R16.2
